Commit message: Update jetbot.urdf

File: src/jetbot_description/urdf/jetbot.urdf (robot description, URDF)
Before this commit: robot JetBot, 7 links, 6 joints
Joints:
- joint right_wheel_hinge: origin xyz=0.03   -0.0595  0.03 rpy=0       0       1.57079 -> xyz=0.03   -0.05125  0.03 rpy=0       0       1.57079

Commit message: Update jetbot.urdf

File: src/jetbot_description/urdf/jetbot.urdf (robot description, URDF)
Before this commit: robot JetBot, 7 links, 6 joints
Joints:
- joint right_wheel_hinge: origin xyz=0.03   -0.05125  0.03 rpy=0       0       1.57079 -> xyz=0.03   -0.059  0.03 rpy=0       0       1.57079
